File: hardware/LoRa-GPS.sch (EAGLE design)
At the start: 27 parts, among them J2 MF-CON-MICROUSB-RIGHT, U1 MCP1703-3302E/CB, Y1 CRYSTAL.ABS07

Commit message: lipo
Parts:
- added C10: 4.7uF, SparkFun-Capacitors:4.7UF-0603-6.3V-(10%)
- added C11: 10uF, SparkFun-Capacitors:10UF-POLAR-EIA3216-16V-10%(TANT)
- added D4: BLUE, SparkFun-LED:LED-BLUE0603
- added J8: (no value), SparkFun-Connectors:CONN_021X02_NO_SILK
- added R5: 2.0k, SparkFun-Resistors:2.0KOHM-0603-1/10W-5%
- added R9: 1k, SparkFun-Resistors:1KOHM-0603-1/10W-1%
- added U2: MCP73831, SparkFun-IC-Power:MCP73831
Connections:
- new net CHARGE_STAT: R9.1, U2.STAT
- new net N$11: R5.1, U2.PROG
- new net N$8: D4.C, R9.2
- new net V_BATT: C11.+, U2.VBAT
- new net V_USB: C10.1, D4.A, J8.2, U2.VIN
- net GND: now also C10.2, C11.-, J8.1, R5.2, U2.VSS
Other:
- note added: "500mA charging"
- note added: "GPS"
- note added: "LIPO CHARGER"
- note added: "RFM95W"
- note added: "SAMD21"
- note added: "USB"
- moved on the sheet: ANT, C1, C2, C3, C4, C5, C6, C7, C8, C9, GPS, J2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
